File: PCB/buck/buck.kicad_pcb (KiCad board)
At the start: 2 copper layers, 30 x 27 mm, 7 parts, among them J1 UBat 38V, J2 Uout 5V, U1 LM2575-5.0BT

Commit message: Add files via upload
Parts:
- added H1: MountingHole_Pad, MountingHole:MountingHole_2.7mm_M2.5_Pad, F.Cu at (149.2, 105.0)
- added H2: MountingHole_Pad, MountingHole:MountingHole_2.7mm_M2.5_Pad, F.Cu at (113.5, 86.0)
- added J3: Zündung, Connector_PinSocket_2.54mm:PinSocket_1x01_P2.54mm_Horizontal, B.Cu at (142.4, 96.0)
- added Q1: QM6006D, Package_TO_SOT_SMD:TO-252-2, B.Cu at (135.0, 96.6)
- added R1: 100k, Resistor_SMD:R_0805_2012Metric, B.Cu at (145.7, 100.1)
- D1: value DIODE -> 1N4148
- J1: footprint Connector_PinHeader_2.00mm:PinHeader_1x02_P2.00mm_Horizontal -> Connector_PinSocket_2.54mm:PinSocket_1x02_P2.54mm_Horizontal; moved to B.Cu
- J2: footprint Connector_PinHeader_2.00mm:PinHeader_1x02_P2.00mm_Vertical -> Connector_PinSocket_2.54mm:PinSocket_1x02_P2.54mm_Horizontal
- moved C2 6.73 mm to (146.4, 88.0)
- moved C1 6.68 mm to (139.8, 105.9)
- moved J2 5.51 mm to (132.2, 91.9), turned to -90 degrees
- moved J1 5.06 mm to (130.5, 101.3), turned to 90 degrees
- moved D1 2.07 mm to (126.7, 97.2)
- moved L1 0.40 mm to (124.1, 89.0)
Connections:
- J1 pad 2: GND -> Net-(J1-Pad2)
Routing:
- net +5V: track 60.7 -> 15.5 mm, vias 0 -> 2
- net Net-(J1-Pad2): track 0.00 -> 24.6 mm
- net Net-(J3-Pad1): track 0.00 -> 8.33 mm
- net Net-(C1-Pad1): track 22.7 -> 20.6 mm
Other:
- board size 30 x 27 mm -> 44.5 x 30 mm

Commit message: Add files via upload
Parts:
- moved R1 11.6 mm to (136.4, 107.1), turned to 180 degrees
- moved C1 8.24 mm to (137.4, 98.0)
- moved J3 5.46 mm to (144.1, 101.2), turned to 90 degrees
- moved Q1 3.72 mm to (137.5, 99.4), turned to 90 degrees
Routing:
- net Net-(J1-Pad2): track 24.6 -> 13.8 mm
- net Net-(C1-Pad1): track 20.6 -> 17.6 mm
- net Net-(J3-Pad1): track 8.33 -> 10.3 mm

Commit message: Add files via upload
Parts:
- moved D1 13.7 mm to (113.2, 99.2), turned to 0 degrees
Routing:
- net +5V: track 15.5 -> 0.00 mm, vias 2 -> 0
Changed lines of the file:
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@@
     (property "Sheetname" "")
     (attr smd)
-    (fp_text reference "C1" (at 5.334 -3.556 180) (layer "F.SilkS")
+    (fp_text reference "C1" (at 5.461 -2.667 180) (layer "F.SilkS")
       (effects (font (size 1 1) (thickness 0.15)))
     )
@@
     (property "Sheetname" "")
     (attr smd)
-    (fp_text reference "C2" (at 4.953 6.604 90) (layer "F.SilkS")
+    (fp_text reference "C2" (at 4.572 6.35) (layer "F.SilkS")
       (effects (font (size 1 1) (thickness 0.15)))
     )
@@
     (property "Sheetname" "")
     (attr smd)
-    (fp_text reference "L1" (at -7.239 5.461 90) (layer "F.SilkS")
+    (fp_text reference "L1" (at -7.239 4.699 180) (layer "F.SilkS")
       (effects (font (size 1 1) (thickness 0.15)))
     )
@@
   )
   (footprint "Diode_SMD:D_0805_2012Metric_Pad1.15x1.40mm_HandSolder" (layer "F.Cu")
-    (at 126.746 97.155 180)
+    (at 113.157 99.187)
     (descr "Diode SMD 0805 (2012 Metric), square (rectangular) end terminal, IPC_7351 nominal, (Body size source: https://docs.google.com/spreadsheets/d/1BsfQQcO9C6DZCsRaXUlFlo91Tg2WpOkGARC1WS5S8t0/edit?usp=sharing), generated with kicad-footprint-generator")
     (tags "diode handsolder")
@@
     (property "Spice_Primitive" "D")
     (attr smd)
-    (fp_text reference "D1" (at 0 -1.65) (layer "F.SilkS")
+    (fp_text reference "D1" (at -1.27 -1.778) (layer "F.SilkS")
       (effects (font (size 1 1) (thickness 0.15)))
     )
@@
     (fp_line (start -0.7 -0.6) (end -1 -0.3) (layer "F.Fab") (width 0.1))
     (fp_line (start 1 0.6) (end 1 -0.6) (layer "F.Fab") (width 0.1))
-    (pad "1" smd roundrect (at -1.025 0 180) (size 1.15 1.4) (layers "F.Cu" "F.Paste" "F.Mask") (roundrect_rratio 0.2173913043)
+    (pad "1" smd roundrect (at -1.025 0) (size 1.15 1.4) (layers "F.Cu" "F.Paste" "F.Mask") (roundrect_rratio 0.2173913043)
       (net 2 "GND") (pinfunction "A") (pintype "passive"))
-    (pad "2" smd roundrect (at 1.025 0 180) (size 1.15 1.4) (layers "F.Cu" "F.Paste" "F.Mask") (roundrect_rratio 0.2173913043)
+    (pad "2" smd roundrect (at 1.025 0) (size 1.15 1.4) (layers "F.Cu" "F.Paste" "F.Mask") (roundrect_rratio 0.2173913043)
       (net 3 "Net-(D1-Pad2)") (pinfunction "K") (pintype "passive"))
     (model "${KICAD6_3DMODEL_DIR}/Diode_SMD.3dshapes/D_0805_2012Metric.wrl"
@@
     (property "Sheetname" "")
     (attr through_hole)
-    (fp_text reference "U1" (at 3.4 -4.27 90) (layer "F.SilkS")
+    (fp_text reference "U1" (at 7.872 -4.167 180) (layer "F.SilkS")
       (effects (font (size 1 1) (thickness 0.15)))
     )
@@
     (property "Sheetname" "")
     (attr smd)
-    (fp_text reference "Q1" (at 4.489 -4.192) (layer "B.SilkS")
+    (fp_text reference "Q1" (at -0.083 3.936) (layer "B.SilkS")
       (effects (font (size 1 1) (thickness 0.15)) (justify mirror))
     )
@@
     (property "Sheetname" "")
     (attr through_hole)
-    (fp_text reference "J1" (at -4.38 2.77 90) (layer "B.SilkS")
+    (fp_text reference "J1" (at -1.225 2.383 180) (layer "B.SilkS")
       (effects (font (size 1 1) (thickness 0.15)) (justify mirror))
     )
@@
     (property "Sheetname" "")
     (attr smd)
-    (fp_text reference "R1" (at 0 1.65) (layer "B.SilkS")
+    (fp_text reference "R1" (at 0 -2.286) (layer "B.SilkS")
       (effects (font (size 1 1) (thickness 0.15)) (justify mirror))
     )
@@
     (property "Sheetname" "")
     (attr through_hole)
-    (fp_text reference "J2" (at -4.38 2.77 90) (layer "B.SilkS")
+    (fp_text reference "J2" (at 0 -4.953) (layer "B.SilkS")
       (effects (font (size 1 1) (thickness 0.15)) (justify mirror))
     )
@@
   (segment (start 130.944 101.264) (end 134.164 98.044) (width 1.5) (layer "F.Cu") (net 1))
   (segment (start 130.459 102.713) (end 130.459 101.264) (width 1.5) (layer "F.Cu") (net 1))
-  (segment (start 121.844 103.2) (end 125.721 99.323) (width 1) (layer "F.Cu") (net 3))
-  (segment (start 125.721 99.323) (end 125.721 97.155) (width 1) (layer "F.Cu") (net 3))
-  (segment (start 120.245 103.2) (end 121.844 103.2) (width 1) (layer "F.Cu") (net 3))
-  (segment (start 119.129 90.563) (end 119.129 89.027) (width 1) (layer "F.Cu") (net 3))
-  (segment (start 125.721 97.155) (end 119.129 90.563) (width 1) (layer "F.Cu") (net 3))
-  (segment (start 129.029 91.824) (end 129.029 89.027) (width 0.75) (layer "F.Cu") (net 4))
-  (segment (start 126.238 94.615) (end 129.029 91.824) (width 0.75) (layer "F.Cu") (net 4))
-  (segment (start 122.069 99.8) (end 120.245 99.8) (width 0.75) (layer "F.Cu") (net 4))
-  (segment (start 122.809 98.425) (end 122.809 99.06) (width 0.75) (layer "F.Cu") (net 4))
-  (segment (start 122.809 99.06) (end 122.069 99.8) (width 0.75) (layer "F.Cu") (net 4))
-  (via (at 122.809 98.425) (size 0.8) (drill 0.4) (layers "F.Cu" "B.Cu") (net 4))
-  (via (at 126.238 94.615) (size 0.8) (drill 0.4) (layers "F.Cu" "B.Cu") (net 4))
-  (segment (start 122.809 98.044) (end 126.238 94.615) (width 0.75) (layer "B.Cu") (net 4))
-  (segment (start 122.809 98.425) (end 122.809 98.044) (width 0.75) (layer "B.Cu") (net 4))
+  (segment (start 114.182 99.187) (end 114.182 92.955) (width 0.8) (layer "F.Cu") (net 3))
+  (segment (start 118.195 103.2) (end 114.182 99.187) (width 0.8) (layer "F.Cu") (net 3))
+  (segment (start 118.11 89.027) (end 119.129 89.027) (width 0.8) (layer "F.Cu") (net 3))
+  (segment (start 120.245 103.2) (end 118.195 103.2) (width 0.8) (layer "F.Cu") (net 3))
+  (segment (start 114.182 92.955) (end 118.11 89.027) (width 0.8) (layer "F.Cu") (net 3))
   (segment (start 137.334 107.061) (end 137.334 106.046) (width 0.75) (layer "B.Cu") (net 5))
   (segment (start 141.351 101.219) (end 144.145 101.219) (width 0.75) (layer "B.Cu") (net 5))
@@
     (polygon
       (pts
-        (xy 141.732 92.837)
-        (xy 127 92.837)
-        (xy 127 84.963)
-        (xy 141.732 84.963)
+        (xy 145.161 93.98)
+        (xy 131.064 93.98)
+        (xy 131.064 98.298)
+        (xy 125.73 98.298)
+        (xy 125.73 100.584)
+        (xy 118.999 100.584)
+        (xy 118.999 96.012)
+        (xy 126.746 96.012)
+        (xy 126.746 84.582)
+        (xy 145.161 84.582)
       )
     )

Commit message: Release v1.0
Parts:
- added R2: 270k, Resistor_SMD:R_0805_2012Metric, B.Cu at (168.9, 104.3)
- added R3: 270k, Resistor_SMD:R_0805_2012Metric, B.Cu at (168.9, 101.2)
- added R4: 30k, Resistor_SMD:R_0805_2012Metric, B.Cu at (168.9, 98.3)
- added R5: 30k, Resistor_SMD:R_0805_2012Metric, B.Cu at (172.1, 99.2)
- added R6: 0R, Resistor_SMD:R_0603_1608Metric, B.Cu at (163.0, 98.3)
- added R7: 0R, Resistor_SMD:R_0603_1608Metric, F.Cu at (155.7, 94.4)
- J2: footprint Connector_PinSocket_2.54mm:PinSocket_1x02_P2.54mm_Horizontal -> Connector_PinSocket_2.54mm:PinSocket_1x03_P2.54mm_Horizontal
- moved R1 23.2 mm to (157.9, 115.8)
- moved Q1 22.2 mm to (157.9, 108.3)
- moved C1 21.9 mm to (158.4, 104.4)
- moved H1 21.9 mm to (170.2, 111.4)
- moved J2 21.9 mm to (153.2, 98.3)
- moved D1 21.9 mm to (134.1, 105.5)
- moved H2 21.9 mm to (134.5, 92.3)
- moved L1 21.9 mm to (145.0, 95.4)
- moved C2 21.9 mm to (167.4, 94.4)
- moved J1 21.9 mm to (151.4, 107.6)
- moved J3 21.9 mm to (165.1, 107.6)
- moved U1 21.9 mm to (141.2, 111.2)
Connections:
- J2 pad 2: +5V -> Net-(J2-Pad2)
Routing:
- net Net-(C1-Pad1): track 17.6 -> 40.3 mm
- net Net-(R3-Pad2): track 0.00 -> 7.09 mm
- net ADC: track 0.00 -> 3.94 mm
- net Net-(J2-Pad2): track 0.00 -> 3.11 mm
- net Net-(R2-Pad2): track 0.00 -> 3.05 mm
- net Net-(R4-Pad2): track 0.00 -> 2.27 mm
- net Net-(J3-Pad1): track 10.3 -> 10.9 mm
- net Net-(J1-Pad2): track 13.8 -> 14.3 mm
