File: PCB/mainboard/mainboard.kicad_sch (KiCad schematic)
At the start: 14 parts

Commit message: Add files via upload
Parts:
- removed C?: F, symbol Device:C
- removed C? (x2): 22pF, symbol Device:C
- removed C?: 100nF, symbol Device:C
- added C1, C2: 22pF, Capacitor_SMD:C_0805_2012Metric, symbol Device:C_Small
- added C4: 100nF, Capacitor_SMD:C_0805_2012Metric, symbol Device:C_Small
- added C5, C6: 100µF, Capacitor_SMD:CP_Elec_5x5.8, symbol Device:C_Polarized_Small
- added C7, C8: 10nF, Capacitor_SMD:C_0603_1608Metric, symbol Device:C_Small
- added H1, H2: MountingHole_Pad, MountingHole:MountingHole_2.7mm_M2.5_Pad, symbol Mechanical:MountingHole_Pad
- added J4: Display, Connector_PinSocket_2.54mm:PinSocket_1x16_P2.54mm_Vertical, symbol Connector:Conn_01x16_Female
- added R6: 0, Resistor_SMD:R_0805_2012Metric, symbol Device:R
- added RV1: Poti, Potentiometer_SMD:Potentiometer_Bourns_3314G_Vertical, symbol Device:R_Potentiometer
- J1: renamed from J?; footprint (none) -> Connector_PinSocket_2.54mm:PinSocket_1x02_P2.54mm_Vertical
- J2, J3: renamed from J?; footprint (none) -> Connector_PinSocket_2.54mm:PinSocket_1x03_P2.54mm_Horizontal
- R1: renamed from R?; value 10k -> 99k; footprint (none) -> Resistor_SMD:R_0805_2012Metric
- R2: renamed from R?; value 82k -> 11k; footprint (none) -> Resistor_SMD:R_0805_2012Metric
- R3: renamed from R?; value R -> 10k; footprint (none) -> Resistor_SMD:R_0805_2012Metric
- R4, R5: renamed from R?; footprint (none) -> Resistor_SMD:R_0805_2012Metric
- Y1: renamed from Y?; value Crystal_Small -> 16MHz; footprint (none) -> Crystal:Crystal_SMD_ECS_CSM3X-2Pin_7.6x4.1mm
- gave numbers to parts that had none: 1
Connections:
- net VBuck is gone; now on net VCC: J2.1 (Pin_1), J3.1 (Pin_1), R1.1, R4.1, R5.1
- net ADC6: now also U1.23 (PC0); no longer U1.19 (ADC6)
- net GND: now also U1.21 (AGND), C1.1, C2.1, C4.2, C5.2, C6.2, C7.2, C8.2, H1.1, H2.1, J4.1 (Pin_1), J4.16 (Pin_16), J4.5 (Pin_5), RV1.1
- net Temp: now also U1.30 (PD0); no longer U1.23 (PC0)
- net VCC: now also J1.2 (Pin_2), C5.1, C6.1, C7.1, C8.1, J4.2 (Pin_2), R6.1, RV1.3
- net at Y1.1: now also U1.8 (PB7/XTAL2), C2.2; no longer U1.7 (PB6/XTAL1)
- net at Y1.2: now also U1.7 (PB6/XTAL1), C1.2; no longer U1.8 (PB7/XTAL2)
- net at R3.2, U1.18 (AVCC): now also C4.1
- new net: J4.15 (Pin_15), R6.2
- new net V0: J4.3 (Pin_3), RV1.2
Other:
- moved on the sheet: J1, J2, J3, R1, R2, R3, R4, R5, U1, Y1

Commit message: Add files via upload
Parts:
- added C3: 100nF, Capacitor_SMD:C_0805_2012Metric, symbol Device:C_Small
- added D1: D, Diode_SMD:D_0805_2012Metric, symbol Device:D
- added R10, R11, R12, R13, R8, R9: 0, Resistor_SMD:R_0805_2012Metric, symbol Device:R
- added R7: 10k, Resistor_SMD:R_0805_2012Metric, symbol Device:R
- added SW1: SW_Push, symbol Switch:SW_Push
Connections:
- net GND: now also C3.1, SW1.1; no longer J4.1 (Pin_1)
- net VCC: now also D1.1 (K), R7.1; no longer J4.2 (Pin_2)
- net at J4.11 (Pin_11): now also R10.1
- net at J4.12 (Pin_12): now also R11.1
- net at J4.13 (Pin_13): now also R12.1
- net at J4.14 (Pin_14): now also R13.2
- net at J4.4 (Pin_4): now also R8.1
- net at J4.6 (Pin_6): now also R9.1
- net PB0: now reaches U1.12 (PB0)
- net PB0: now also R8.2
- net PB1: now reaches U1.13 (PB1)
- net PB1: now also R9.2
- net PB2: now reaches U1.14 (PB2)
- net PB2: now also R10.2
- net PB3: now reaches U1.15 (PB3)
- net PB3: now also R11.2
- net PB4: now reaches U1.16 (PB4)
- net PB4: now also R12.2
- net PB5: now reaches U1.17 (PB5)
- net PB5: now also R13.1
- net RESET: now reaches U1.29 (PC6/~{RESET})
- net RESET: now also C3.2, D1.2 (A), R7.2, SW1.2
- new net Vdd: J4.2 (Pin_2)
- new net Vss: J4.1 (Pin_1)
- no-connect marks 0 -> 15

Commit message: Add files via upload
Parts:
- SW1: footprint (none) -> Button_Switch_THT:SW_PUSH_6mm
Connections:
- net Vss is gone; now on net GND: J4.1 (Pin_1)
Changed lines of the file:
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@@
+    (stroke (width 0) (type default) (color 0 0 0 0))
+  )
+  (wire (pts (xy 157.48 102.87) (xy 149.86 102.87))
     (stroke (width 0) (type default) (color 0 0 0 0))
   )
@@
   )
   (wire (pts (xy 48.26 55.88) (xy 55.88 55.88))
-    (stroke (width 0) (type default) (color 0 0 0 0))
-  )
-  (wire (pts (xy 152.4 102.87) (xy 157.48 102.87))
     (stroke (width 0) (type default) (color 0 0 0 0))
   )
@@
     (effects (font (size 1 1)) (justify right))
     (property "Intersheet References" "${INTERSHEET_REFS}" (id 0) (at 77.3962 71.0575 0)
-      (effects (font (size 1 1)) (justify right) hide)
-    )
-  )
-  (global_label "Vss" (shape output) (at 152.4 102.87 180) (fields_autoplaced)
-    (effects (font (size 1 1)) (justify right))
-    (property "Intersheet References" "${INTERSHEET_REFS}" (id 0) (at 148.0238 102.8075 0)
       (effects (font (size 1 1)) (justify right) hide)
     )
@@
     )
     (property "Datasheet" "" (id 3) (at 72.39 129.54 0)
+      (effects (font (size 1.27 1.27)) hide)
+    )
+    (pin "1")
+  )
+  (symbol (lib_id "power:GND") (at 149.86 102.87 270) (unit 1)
+    (in_bom yes) (on_board yes) (fields_autoplaced)
+    (property "Reference" "#PWR0123" (id 0) (at 143.51 102.87 0)
+      (effects (font (size 1.27 1.27)) hide)
+    )
+    (property "Value" "GND" (id 1) (at 144.78 102.87 0))
+    (property "Footprint" "" (id 2) (at 149.86 102.87 0)
+      (effects (font (size 1.27 1.27)) hide)
+    )
+    (property "Datasheet" "" (id 3) (at 149.86 102.87 0)
       (effects (font (size 1.27 1.27)) hide)
     )
@@
       (effects (font (size 1.27 1.27)) (justify right))
     )
-    (property "Footprint" "" (id 2) (at 27.94 96.52 0)
+    (property "Footprint" "Button_Switch_THT:SW_PUSH_6mm" (id 2) (at 27.94 96.52 0)
       (effects (font (size 1.27 1.27)) hide)
     )
@@
       (reference "#PWR0122") (unit 1) (value "VCC") (footprint "")
     )
+    (path "/69946b56-2cb4-469a-a310-d0d2fdc38279"
+      (reference "#PWR0123") (unit 1) (value "GND") (footprint "")
+    )
     (path "/5ee03960-7870-4430-a073-e90b29c25f62"
       (reference "C1") (unit 1) (value "22pF") (footprint "Capacitor_SMD:C_0805_2012Metric")
@@
     )
     (path "/ebee871f-2694-4148-af27-f7cd2d5b559e"
-      (reference "SW1") (unit 1) (value "SW_Push") (footprint "")
+      (reference "SW1") (unit 1) (value "SW_Push") (footprint "Button_Switch_THT:SW_PUSH_6mm")
     )
     (path "/ce5ceab1-5f31-44b1-aa53-18904ee5a322"

Commit message: PCB error correction
Connections:
- net Vdd is gone; now on net VCC: J4.2 (Pin_2)
- no-connect marks 15 -> 14
Changed lines of the file:
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@@
   (junction (at 55.88 55.88) (diameter 0) (color 0 0 0 0)
   )
+  (junction (at 71.12 55.88) (diameter 0) (color 0 0 0 0)
+  )
   (junction (at 189.23 83.82) (diameter 0) (color 0 0 0 0)
   )
+  (junction (at 71.12 45.72) (diameter 0) (color 0 0 0 0)
+  )
   (junction (at 33.02 88.9) (diameter 0) (color 0 0 0 0)
   )
@@
   )
   (no_connect (at 86.36 91.44))
-  (no_connect (at 86.36 71.12))
   (no_connect (at 116.84 109.22))
   (no_connect (at 116.84 93.98))
@@
     (stroke (width 0) (type default) (color 0 0 0 0))
   )
+  (wire (pts (xy 71.12 44.45) (xy 71.12 45.72))
+    (stroke (width 0) (type default) (color 0 0 0 0))
+  )
   (wire (pts (xy 142.24 138.43) (xy 142.24 139.7))
     (stroke (width 0) (type default) (color 0 0 0 0))
@@
     (stroke (width 0) (type default) (color 0 0 0 0))
   )
+  (wire (pts (xy 99.695 55.88) (xy 104.14 55.88))
+    (stroke (width 0) (type default) (color 0 0 0 0))
+  )
   (wire (pts (xy 104.14 44.45) (xy 104.14 45.72))
     (stroke (width 0) (type default) (color 0 0 0 0))
@@
   )
   (wire (pts (xy 194.31 72.39) (xy 194.31 74.93))
+    (stroke (width 0) (type default) (color 0 0 0 0))
+  )
+  (wire (pts (xy 71.12 55.88) (xy 71.12 57.15))
     (stroke (width 0) (type default) (color 0 0 0 0))
   )
@@
   )
   (label "PB0" (at 124.46 71.12 0)
+    (effects (font (size 1.27 1.27)) (justify left bottom))
+  )
+  (label "{PB0 PB1 PB2 PB3 PB4 PB5}" (at 134.62 120.015 90)
     (effects (font (size 1.27 1.27)) (justify left bottom))
   )
@@
     )
   )
-  (global_label "Vdd" (shape output) (at 152.4 105.41 180) (fields_autoplaced)
-    (effects (font (size 1 1)) (justify right))
-    (property "Intersheet References" "${INTERSHEET_REFS}" (id 0) (at 147.8333 105.3475 0)
-      (effects (font (size 1 1)) (justify right) hide)
-    )
-  )
   (global_label "V0" (shape output) (at 177.8 115.57 180) (fields_autoplaced)
     (effects (font (size 1 1)) (justify right))
@@
     (pin "1")
   )
+  (symbol (lib_id "power:VCC") (at 152.4 105.41 90) (unit 1)
+    (in_bom yes) (on_board yes) (fields_autoplaced)
+    (property "Reference" "#PWR0124" (id 0) (at 156.21 105.41 0)
+      (effects (font (size 1.27 1.27)) hide)
+    )
+    (property "Value" "VCC" (id 1) (at 153.67 105.4099 90)
+      (effects (font (size 1.27 1.27)) (justify right))
+    )
+    (property "Footprint" "" (id 2) (at 152.4 105.41 0)
+      (effects (font (size 1.27 1.27)) hide)
+    )
+    (property "Datasheet" "" (id 3) (at 152.4 105.41 0)
+      (effects (font (size 1.27 1.27)) hide)
+    )
+    (pin "1")
+  )
   (symbol (lib_id "power:GND") (at 101.6 137.16 0) (unit 1)
     (in_bom yes) (on_board yes) (fields_autoplaced)
@@
     )
     (property "Datasheet" "" (id 3) (at 101.6 137.16 0)
+      (effects (font (size 1.27 1.27)) hide)
+    )
+    (pin "1")
+  )
+  (symbol (lib_id "power:PWR_FLAG") (at 99.695 55.88 90) (unit 1)
+    (in_bom yes) (on_board yes) (fields_autoplaced)
+    (property "Reference" "#FLG0102" (id 0) (at 97.79 55.88 0)
+      (effects (font (size 1.27 1.27)) hide)
+    )
+    (property "Value" "PWR_FLAG" (id 1) (at 96.52 55.8799 90)
+      (effects (font (size 1.27 1.27)) (justify left))
+    )
+    (property "Footprint" "" (id 2) (at 99.695 55.88 0)
+      (effects (font (size 1.27 1.27)) hide)
+    )
+    (property "Datasheet" "~" (id 3) (at 99.695 55.88 0)
       (effects (font (size 1.27 1.27)) hide)
     )
@@
     (pin "2")
   )
+  (symbol (lib_id "power:PWR_FLAG") (at 71.12 44.45 0) (unit 1)
+    (in_bom yes) (on_board yes) (fields_autoplaced)
+    (property "Reference" "#FLG0101" (id 0) (at 71.12 42.545 0)
+      (effects (font (size 1.27 1.27)) hide)
+    )
+    (property "Value" "PWR_FLAG" (id 1) (at 71.12 39.37 0))
+    (property "Footprint" "" (id 2) (at 71.12 44.45 0)
+      (effects (font (size 1.27 1.27)) hide)
+    )
+    (property "Datasheet" "~" (id 3) (at 71.12 44.45 0)
+      (effects (font (size 1.27 1.27)) hide)
+    )
+    (pin "1")
+  )
   (symbol (lib_id "power:VCC") (at 194.31 72.39 0) (unit 1)
     (in_bom yes) (on_board yes) (fields_autoplaced)
@@
     )
     (property "Datasheet" "" (id 3) (at 55.88 57.15 0)
+      (effects (font (size 1.27 1.27)) hide)
+    )
+    (pin "1")
+  )
+  (symbol (lib_id "power:PWR_FLAG") (at 71.12 57.15 180) (unit 1)
+    (in_bom yes) (on_board yes) (fields_autoplaced)
+    (property "Reference" "#FLG0103" (id 0) (at 71.12 59.055 0)
+      (effects (font (size 1.27 1.27)) hide)
+    )
+    (property "Value" "PWR_FLAG" (id 1) (at 71.12 61.595 0))
+    (property "Footprint" "" (id 2) (at 71.12 57.15 0)
+      (effects (font (size 1.27 1.27)) hide)
+    )
+    (property "Datasheet" "~" (id 3) (at 71.12 57.15 0)
       (effects (font (size 1.27 1.27)) hide)
     )
@@
   )
   (symbol_instances
+    (path "/2d7815f3-1326-48ca-83ef-dd4678e6f521"
+      (reference "#FLG0101") (unit 1) (value "PWR_FLAG") (footprint "")
+    )
+    (path "/0ee8841b-c906-474e-baf5-133a38486fcb"
+      (reference "#FLG0102") (unit 1) (value "PWR_FLAG") (footprint "")
+    )
+    (path "/76318992-0309-4787-aabd-6ad03a28e02b"
+      (reference "#FLG0103") (unit 1) (value "PWR_FLAG") (footprint "")
+    )
     (path "/640f687d-1436-449a-839e-643c7523961d"
       (reference "#PWR0101") (unit 1) (value "GND") (footprint "")
@@
       (reference "#PWR0123") (unit 1) (value "GND") (footprint "")
     )
+    (path "/0e6a33cc-9e8f-4714-9458-e5bdf7d277ad"
+      (reference "#PWR0124") (unit 1) (value "VCC") (footprint "")
+    )
     (path "/5ee03960-7870-4430-a073-e90b29c25f62"

Commit message: Release v1.0
Parts:
- removed R1: 99k, Resistor_SMD:R_0805_2012Metric, symbol Device:R
- removed R2: 11k, Resistor_SMD:R_0805_2012Metric, symbol Device:R
- J1: footprint Connector_PinSocket_2.54mm:PinSocket_1x02_P2.54mm_Vertical -> Connector_PinSocket_2.54mm:PinSocket_1x03_P2.54mm_Vertical; symbol Connector:Conn_01x02_Female -> Connector:Conn_01x03_Female
Connections:
- net ADC6: now also J1.2 (Pin_2)
- net VCC: now also J1.3 (Pin_3); no longer J1.2 (Pin_2)
Other:
- moved on the sheet: C3, SW1
